File: pcb/Breakouts/Keg Cop - Daisy Chain.sch (EAGLE design)
At the start: 3 parts, among them X1 RJ45-8X, X2 RJ45-8X

Commit message: Rename files
Parts:
- FLOW: value 3-PIN -> (none); device Donnie:HDR-3 -> con-wago-500:W237-103
- renumbered X1 to IN, X2 to OUT
Connections:
- removed net FLOW: FLOW.2, IN.1
- new net DATA: FLOW-2.KL, IN.1
- net 5V: now also FLOW-1.KL; no longer FLOW.3
- net GND: now also FLOW-3.KL; no longer FLOW.1
Changed lines of the file:
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@@
 </classes>
 <parts>
-<part name="X1" library="con-tycoelectronics" library_urn="urn:adsk.eagle:library:193" deviceset="RJ45" device="" package3d_urn="urn:adsk.eagle:package:10660/1" technology="-8X"/>
-<part name="X2" library="con-tycoelectronics" library_urn="urn:adsk.eagle:library:193" deviceset="RJ45" device="" package3d_urn="urn:adsk.eagle:package:10660/1" technology="-8X"/>
-<part name="FLOW" library="Donnie" deviceset="HDR-3" device="" value="3-PIN"/>
+<part name="IN" library="con-tycoelectronics" library_urn="urn:adsk.eagle:library:193" deviceset="RJ45" device="" package3d_urn="urn:adsk.eagle:package:10660/1" technology="-8X"/>
+<part name="OUT" library="con-tycoelectronics" library_urn="urn:adsk.eagle:library:193" deviceset="RJ45" device="" package3d_urn="urn:adsk.eagle:package:10660/1" technology="-8X"/>
+<part name="FLOW" library="con-wago-500" library_urn="urn:adsk.eagle:library:195" deviceset="W237-103" device="" package3d_urn="urn:adsk.eagle:package:10691/1"/>
 </parts>
 <sheets>
@@
 </plain>
 <instances>
-<instance part="X1" gate="G$1" x="63.5" y="33.02" smashed="yes" rot="R270">
+<instance part="IN" gate="G$1" x="63.5" y="33.02" smashed="yes" rot="R270">
 <attribute name="NAME" x="73.66" y="35.56" size="1.778" layer="95" rot="R270"/>
 <attribute name="VALUE" x="50.292" y="35.56" size="1.778" layer="96" rot="R270"/>
 </instance>
-<instance part="X2" gate="G$1" x="60.96" y="68.58" smashed="yes" rot="R90">
+<instance part="OUT" gate="G$1" x="60.96" y="68.58" smashed="yes" rot="R90">
 <attribute name="NAME" x="50.8" y="66.04" size="1.778" layer="95" rot="R90"/>
 <attribute name="VALUE" x="74.168" y="66.04" size="1.778" layer="96" rot="R90"/>
 </instance>
-<instance part="FLOW" gate="G$1" x="96.52" y="53.34" smashed="yes" rot="R180">
-<attribute name="VALUE" x="97.79" y="58.42" size="1.778" layer="96" rot="R180"/>
-<attribute name="NAME" x="97.79" y="44.958" size="1.778" layer="95" rot="R180"/>
+<instance part="FLOW" gate="-1" x="93.98" y="55.88" smashed="yes" rot="R180">
+<attribute name="NAME" x="93.98" y="54.991" size="1.778" layer="95"/>
+</instance>
+<instance part="FLOW" gate="-2" x="93.98" y="50.8" smashed="yes" rot="R180">
+<attribute name="NAME" x="93.98" y="49.911" size="1.778" layer="95"/>
+</instance>
+<instance part="FLOW" gate="-3" x="93.98" y="45.72" smashed="yes" rot="R180">
+<attribute name="VALUE" x="96.52" y="49.403" size="1.778" layer="96" rot="R180"/>
+<attribute name="NAME" x="93.98" y="44.831" size="1.778" layer="95"/>
 </instance>
 </instances>
@@
 <net name="GND" class="0">
 <segment>
-<pinref part="X1" gate="G$1" pin="8"/>
+<pinref part="FLOW" gate="-3" pin="KL"/>
+<label x="83.82" y="45.72" size="1.778" layer="95"/>
+<pinref part="IN" gate="G$1" pin="8"/>
 <wire x1="53.34" y1="35.56" x2="53.34" y2="50.8" width="0.1524" layer="91"/>
-<pinref part="X2" gate="G$1" pin="8"/>
-<wire x1="71.12" y1="50.8" x2="71.12" y2="53.34" width="0.1524" layer="91"/>
-<wire x1="71.12" y1="53.34" x2="71.12" y2="66.04" width="0.1524" layer="91"/>
+<pinref part="OUT" gate="G$1" pin="8"/>
+<wire x1="71.12" y1="50.8" x2="71.12" y2="66.04" width="0.1524" layer="91"/>
 <wire x1="53.34" y1="50.8" x2="71.12" y2="50.8" width="0.1524" layer="91"/>
-<pinref part="FLOW" gate="G$1" pin="1"/>
-<wire x1="88.9" y1="53.34" x2="71.12" y2="53.34" width="0.1524" layer="91"/>
-<junction x="71.12" y="53.34"/>
-<label x="83.82" y="53.34" size="1.778" layer="95"/>
+<wire x1="71.12" y1="50.8" x2="71.12" y2="45.72" width="0.1524" layer="91"/>
+<junction x="71.12" y="50.8"/>
+<wire x1="88.9" y1="45.72" x2="71.12" y2="45.72" width="0.1524" layer="91"/>
 </segment>
 </net>
 <net name="5V" class="0">
 <segment>
-<pinref part="X1" gate="G$1" pin="7"/>
+<pinref part="IN" gate="G$1" pin="7"/>
 <wire x1="55.88" y1="35.56" x2="55.88" y2="48.26" width="0.1524" layer="91"/>
-<pinref part="X2" gate="G$1" pin="7"/>
-<wire x1="68.58" y1="48.26" x2="68.58" y2="66.04" width="0.1524" layer="91"/>
+<pinref part="OUT" gate="G$1" pin="7"/>
+<wire x1="68.58" y1="48.26" x2="68.58" y2="55.88" width="0.1524" layer="91"/>
+<wire x1="68.58" y1="55.88" x2="68.58" y2="66.04" width="0.1524" layer="91"/>
 <wire x1="55.88" y1="48.26" x2="68.58" y2="48.26" width="0.1524" layer="91"/>
-<pinref part="FLOW" gate="G$1" pin="3"/>
-<wire x1="68.58" y1="48.26" x2="88.9" y2="48.26" width="0.1524" layer="91"/>
-<junction x="68.58" y="48.26"/>
-<label x="83.82" y="48.26" size="1.778" layer="95"/>
+<junction x="68.58" y="55.88"/>
+<pinref part="FLOW" gate="-1" pin="KL"/>
+<label x="83.82" y="55.88" size="1.778" layer="95"/>
+<wire x1="68.58" y1="55.88" x2="88.9" y2="55.88" width="0.1524" layer="91"/>
 </segment>
 </net>
 <net name="N$1" class="0">
 <segment>
-<pinref part="X1" gate="G$1" pin="2"/>
+<pinref part="IN" gate="G$1" pin="2"/>
 <wire x1="68.58" y1="35.56" x2="68.58" y2="45.72" width="0.1524" layer="91"/>
 <wire x1="68.58" y1="45.72" x2="58.42" y2="45.72" width="0.1524" layer="91"/>
 <wire x1="58.42" y1="45.72" x2="58.42" y2="53.34" width="0.1524" layer="91"/>
 <wire x1="58.42" y1="53.34" x2="53.34" y2="53.34" width="0.1524" layer="91"/>
-<pinref part="X2" gate="G$1" pin="1"/>
+<pinref part="OUT" gate="G$1" pin="1"/>
 <wire x1="53.34" y1="53.34" x2="53.34" y2="66.04" width="0.1524" layer="91"/>
 </segment>
@@
 <net name="N$2" class="0">
 <segment>
-<pinref part="X2" gate="G$1" pin="2"/>
+<pinref part="OUT" gate="G$1" pin="2"/>
 <wire x1="55.88" y1="66.04" x2="55.88" y2="55.88" width="0.1524" layer="91"/>
 <wire x1="55.88" y1="55.88" x2="66.04" y2="55.88" width="0.1524" layer="91"/>
-<pinref part="X1" gate="G$1" pin="3"/>
+<pinref part="IN" gate="G$1" pin="3"/>
 <wire x1="66.04" y1="55.88" x2="66.04" y2="35.56" width="0.1524" layer="91"/>
 </segment>
@@
 <net name="N$3" class="0">
 <segment>
-<pinref part="X1" gate="G$1" pin="4"/>
+<pinref part="IN" gate="G$1" pin="4"/>
 <wire x1="63.5" y1="35.56" x2="63.5" y2="58.42" width="0.1524" layer="91"/>
 <wire x1="63.5" y1="58.42" x2="58.42" y2="58.42" width="0.1524" layer="91"/>
-<pinref part="X2" gate="G$1" pin="3"/>
+<pinref part="OUT" gate="G$1" pin="3"/>
 <wire x1="58.42" y1="58.42" x2="58.42" y2="66.04" width="0.1524" layer="91"/>
 </segment>
@@
 <net name="N$5" class="0">
 <segment>
-<pinref part="X1" gate="G$1" pin="5"/>
-<pinref part="X2" gate="G$1" pin="4"/>
+<pinref part="IN" gate="G$1" pin="5"/>
+<pinref part="OUT" gate="G$1" pin="4"/>
 <wire x1="60.96" y1="35.56" x2="60.96" y2="66.04" width="0.1524" layer="91"/>
 </segment>
@@
 <net name="N$7" class="0">
 <segment>
-<pinref part="X1" gate="G$1" pin="6"/>
+<pinref part="IN" gate="G$1" pin="6"/>
 <wire x1="58.42" y1="35.56" x2="58.42" y2="43.18" width="0.1524" layer="91"/>
 <wire x1="58.42" y1="43.18" x2="50.8" y2="43.18" width="0.1524" layer="91"/>
 <wire x1="50.8" y1="43.18" x2="50.8" y2="60.96" width="0.1524" layer="91"/>
 <wire x1="50.8" y1="60.96" x2="63.5" y2="60.96" width="0.1524" layer="91"/>
-<pinref part="X2" gate="G$1" pin="5"/>
+<pinref part="OUT" gate="G$1" pin="5"/>
 <wire x1="63.5" y1="60.96" x2="63.5" y2="66.04" width="0.1524" layer="91"/>
 </segment>
 </net>
-<net name="FLOW" class="0">
+<net name="DATA" class="0">
 <segment>
-<pinref part="X1" gate="G$1" pin="1"/>
+<pinref part="FLOW" gate="-2" pin="KL"/>
+<label x="83.82" y="50.8" size="1.778" layer="95"/>
+<pinref part="IN" gate="G$1" pin="1"/>
 <wire x1="71.12" y1="35.56" x2="71.12" y2="38.1" width="0.1524" layer="91"/>
-<wire x1="71.12" y1="38.1" x2="76.2" y2="38.1" width="0.1524" layer="91"/>
-<wire x1="76.2" y1="38.1" x2="76.2" y2="50.8" width="0.1524" layer="91"/>
-<pinref part="FLOW" gate="G$1" pin="2"/>
-<wire x1="76.2" y1="50.8" x2="88.9" y2="50.8" width="0.1524" layer="91"/>
-<label x="83.82" y="50.8" size="1.778" layer="95"/>
+<wire x1="73.66" y1="50.8" x2="73.66" y2="38.1" width="0.1524" layer="91"/>
+<wire x1="73.66" y1="38.1" x2="71.12" y2="38.1" width="0.1524" layer="91"/>
+<wire x1="88.9" y1="50.8" x2="73.66" y2="50.8" width="0.1524" layer="91"/>
 </segment>
 </net>
