File: pcb/Main Boards/Keg Cop.sch (EAGLE design)
At the start: 14 parts, among them X1 RJ45-8X, X2 RJ45-8X

Commit message: Rename files
Parts:
- added ROOM: 3-PIN, Donnie:HDR-3
Connections:
- new net KEG7: D32.IO22, X2.7
- new net KEG8: D32.IO23, X2.8
- net 5V: now also ROOM.2; no longer X2.7
- net COOL: now also RELAY.2; no longer RELAY.3
- net GND: now also ROOM.1; no longer X2.8
- net RDAT: now also ROOM.3
- net SOL: now also RELAY.3; no longer RELAY.2
Other:
- moved on the sheet: C1, C2, C3, C4, D32, POWER, R1, R2, R3, R4, R5, RELAY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
