File: pcb/Main Boards/Keg Cop.brd (EAGLE design)
At the start: 65 x 51 mm, 17 parts, among them X1 RJ45-8X, X2 RJ45-8X

Commit message: Rename files
Parts:
- added ROOM: 3-PIN, Donnie:HDR-3_VERT
- moved U$1 2.80 mm to (4.50, 33.0)
- moved POWER 0.54 mm to (9.71, 42.0)
- moved RELAY 0.50 mm to (13.5, 47.4)
Connections:
- net 5V: now also ROOM.2
- net GND: now also ROOM.1
- net RDAT: now also ROOM.3
Routing:
- net RDAT: track 38.9 -> 42.8 mm
- net TDAT: track 31.8 -> 30.9 mm
- net 3V3: track 40.1 -> 39.4 mm
- net COOL: track 33.7 -> 33.1 mm
- net LDAT: track 26.6 -> 26.1 mm
Other:
- board text added: "D"

Commit message: Update images
Parts:
- moved U$1 1.00 mm to (4.50, 32.0)
Changed lines of the file:
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@@
 <?xml version="1.0" encoding="utf-8"?>
 <!DOCTYPE eagle SYSTEM "eagle.dtd">
-<eagle version="9.5.2">
+<eagle version="9.6.1">
 <drawing>
 <settings>
@@
 <attribute name="NAME" x="25.435" y="14.03" size="0.8128" layer="25" align="center-right"/>
 </element>
-<element name="U$1" library="holes" library_urn="urn:adsk.eagle:library:237" package="3,0" package3d_urn="urn:adsk.eagle:package:14277/1" value="" x="4.5" y="33" smashed="yes"/>
+<element name="U$1" library="holes" library_urn="urn:adsk.eagle:library:237" package="3,0" package3d_urn="urn:adsk.eagle:package:14277/1" value="" x="4.5" y="32" smashed="yes"/>
 <element name="U$2" library="holes" library_urn="urn:adsk.eagle:library:237" package="3,0" package3d_urn="urn:adsk.eagle:package:14277/1" value="" x="32.5" y="4.5" smashed="yes"/>
 <element name="U$3" library="holes" library_urn="urn:adsk.eagle:library:237" package="3,0" package3d_urn="urn:adsk.eagle:package:14277/1" value="" x="60.5" y="46.5" smashed="yes"/>
@@
 <wire x1="22.3" y1="9.6" x2="23.8" y2="11.1" width="1.016" layer="1"/>
 <wire x1="23.8" y1="11.1" x2="28.8" y2="11.1" width="1.016" layer="1"/>
-<wire x1="2.4" y1="11.28975" x2="2.4" y2="23.6" width="1.016" layer="16"/>
+<wire x1="2.4" y1="11.28975" x2="2.4" y2="23.4" width="1.016" layer="16"/>
 <wire x1="2.4" y1="11.28975" x2="5.48975" y2="8.2" width="1.016" layer="16"/>
 <wire x1="13.175" y1="10.375" x2="13.175" y2="11.85" width="1.016" layer="16"/>
@@
 <wire x1="9.707" y1="36.4" x2="9.707" y2="36.6" width="1.016" layer="16"/>
 <wire x1="9.707" y1="36.6" x2="9.707" y2="42" width="1.016" layer="16"/>
-<wire x1="9.707" y1="30.907" x2="9.707" y2="36.6" width="1.016" layer="16"/>
-<wire x1="2.4" y1="23.6" x2="9.707" y2="30.907" width="1.016" layer="16"/>
+<wire x1="9.707" y1="30.707" x2="9.707" y2="36.4" width="1.016" layer="16"/>
+<wire x1="2.4" y1="23.4" x2="9.707" y2="30.707" width="1.016" layer="16"/>
 </signal>
 <signal name="RDAT">
