File: pcb/Main Boards/Keg Cop - New 8-Pack.brd (EAGLE design)
At the start: 65 x 51 mm, 18 parts, among them X1 RJ45-8X, X2 RJ45-8X

Commit message: Begin new board for 8 flowmeters
Parts:
- added FLOW1-4: RJ45-8X, con-tycoelectronics:RJ45-NO-SHIELD
- added IC1: DS18B20+, SamacSys_Parts:TO-92
- moved U$3 20.5 mm to (81.0, 46.5)
- moved ROOM 1.53 mm to (10.7, 35.2)
- moved POWER 1.20 mm to (10.7, 41.3)
- moved RELAY 1.01 mm to (14.5, 47.5)
- moved U$1 1.00 mm to (4.50, 33.0)
- renumbered X1 to SENSORS, X2 to FLOW5-8
Connections:
- net 5V: now also FLOW1-4.7, FLOW5-8.7, IC1.3
- net COOL: now also RELAY.3; no longer RELAY.2
- net GND: now also FLOW1-4.8, FLOW5-8.8, IC1.1
- net KEG5: now also FLOW1-4.1; no longer FLOW5-8.5
- net KEG6: now also FLOW1-4.2; no longer FLOW5-8.6
- net KEG7: now also FLOW1-4.3; no longer FLOW5-8.7
- net KEG8: now also FLOW1-4.4; no longer FLOW5-8.8
- net RDAT: now also IC1.2
- net SOL: now also RELAY.2; no longer RELAY.3
Routing:
- net GND: track 175.1 -> 320.5 mm
- net 5V: track 44.2 -> 117.5 mm
- net RDAT: track 42.8 -> 60.8 mm
- net COOL: track 33.1 -> 24.0 mm
- net KEG6: track 30.5 -> 37.3 mm
- net KEG8: track 40.8 -> 47.0 mm
- net KEG7: track 43.9 -> 49.9 mm
- net SOL: track 75.6 -> 78.7 mm
- net 3V3: track 39.4 -> 38.1 mm
- net KEG5: track 36.6 -> 36.0 mm
Other:
- board size 65 x 51 mm -> 85 x 51 mm
- board text added: "1 - FLOW1 2 - FLOW2 3 - FLOW3 4 - FLOW4"
- board text added: "1 - FLOW5 2 - FLOW6 3 - FLOW7 4 - FLOW8"
- board text added: "1 - RDAT 2 - TDAT 3 - UDAT 4 - LDAT"
- board text added: "7 - 5V 8 - GND"
- board text removed: "5 - KEG5 6 - KEG6 7 - KEG7 8 - KEG8"
- board text removed: "X1 1 - RDAT 2 - TDAT 3 - UDAT 4 - LDAT"
- board text removed: "X2 1 - KEG1 2 - KEG2 3 - KEG3 4 - KEG4"
