File: pcb/Breakouts/sensors/Keg Cop - Sensors.brd (EAGLE design)
At the start: 36.6 x 33.3 mm, 6 parts

Commit message: Organize files
Parts:
- moved KDAT 4.60 mm to (35.6, 7.60)
- moved LDAT 4.60 mm to (35.6, 25.7)
- moved TDAT 4.60 mm to (1.00, 25.7)
- moved UDAT 4.60 mm to (1.00, 7.60)
Routing:
- net 5V: track 82.8 -> 94.4 mm
- net GND: track 81.6 -> 91.6 mm
- net TDAT: track 14.8 -> 19.4 mm
- net UDAT: track 18.5 -> 22.8 mm
- net KDAT: track 19.4 -> 23.2 mm
- net LDAT: track 27.0 -> 28.9 mm
- added copper zone on layer 1, net GND
- added copper zone on layer 16, net GND
Other:
- board size 36.6 x 33.3 mm -> 45.8 x 33.3 mm
