File: pcb/Main Boards/devel/Keg Cop - Devel TH.sch (EAGLE design)
At the start: 25 parts

Commit message: Demo board (#91)
* New TH design

* New TH design

* New SMD design
Parts:
- added C3: 0.1μF, Donnie:CAP_CERAMIC_2.54
- added C4: 1.0μF, Donnie:CAP_CERAMIC_2.54
- added FLOW8: (no value), switch-omron:10-XX
- added R10, R11, R12, R13, R14, R15, R16, R8, R9: 2.2kΩ, SparkFun-Resistors:RESISTORAXIAL-0.3
- D32: SPICEPREFIX (none) -> X
Connections:
- removed net KEG1: D32.IO0, FLOW0.P
- removed net KEG2: D32.IO4, FLOW1.P
- removed net KEG3: D32.IO17, FLOW2.P
- removed net KEG4: D32.IO18, FLOW3.P
- removed net KEG5: D32.IO19, FLOW4.P
- removed net KEG6: D32.IO21, FLOW5.P
- removed net KEG7: D32.IO22, FLOW6.P
- removed net KEG8: D32.IO23, FLOW7.P
- new net FLOW0: D32.IO4, FLOW0.S, FLOW0.S1, R8.2
- new net FLOW1: D32.IO16, FLOW1.S, FLOW1.S1, R9.2
- new net FLOW2: D32.IO17, FLOW2.S, FLOW2.S1, R10.2
- new net FLOW3: D32.IO18, FLOW3.S, FLOW3.S1, R11.2
- new net FLOW4: D32.IO19, FLOW4.S, FLOW4.S1, R12.2
- new net FLOW5: D32.IO21, FLOW5.S, FLOW5.S1, R13.2
- new net FLOW6: D32.IO22, FLOW6.S, FLOW6.S1, R14.2
- new net FLOW7: D32.IO23, FLOW7.S, FLOW7.S1, R15.2
- new net FLOW8: D32.IO13, FLOW8.S, FLOW8.S1, R16.2
- new net VBUS: C3.2, C4.2, D32.VBUS
- net 3V3: now also R10.1, R11.1, R12.1, R13.1, R14.1, R15.1, R16.1, R8.1, R9.1
- net GND: now also C3.1, C4.1, FLOW0.P, FLOW0.P1, FLOW1.P, FLOW1.P1, FLOW2.P, FLOW2.P1, FLOW3.P, FLOW3.P1, FLOW4.P, FLOW4.P1, FLOW5.P, FLOW5.P1, FLOW6.P, FLOW6.P1, FLOW7.P, FLOW7.P1, FLOW8.P, FLOW8.P1; no longer FLOW0.S, FLOW1.S, FLOW2.S, FLOW3.S, FLOW4.S, FLOW5.S, FLOW6.S, FLOW7.S
- net N$1: now also R6.2; no longer R7.2
- net N$2: now also R7.2; no longer R6.2
- net SOL: now also D32.IO2; no longer D32.IO16
Other:
- moved on the sheet: C1, C2, COOL, D32, FLOW0, FLOW1, FLOW2, FLOW3, FLOW4, FLOW5, FLOW6, FLOW7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
