File: pcb/Main Boards/devel/SMD/Keg Cop - Devel SMD.sch (EAGLE design)
At the start: 37 parts

Commit message: Organize and order SMD
Parts:
- R10, R11: value 2k2Ω -> 60.4Ω
Changed lines of the file:
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@@
 <part name="SOLENOID" library="JBJLC" deviceset="LED_0603" device="LED_SMD_0603"/>
 <part name="COOL" library="JBJLC" deviceset="LED_0603" device="LED_SMD_0603"/>
-<part name="R11" library="JBJLC" deviceset="RES_SMD" device="0805" value="2k2Ω"/>
+<part name="R11" library="JBJLC" deviceset="RES_SMD" device="0805" value="60.4Ω"/>
 <part name="KEG" library="JBJLC" deviceset="DS18B20Z" device=""/>
 <part name="LOWER" library="JBJLC" deviceset="DS18B20Z" device=""/>
@@
 <part name="TOWER" library="JBJLC" deviceset="DS18B20Z" device=""/>
 <part name="ROOM" library="JBJLC" deviceset="DS18B20Z" device=""/>
-<part name="R10" library="JBJLC" deviceset="RES_SMD" device="0805" value="2k2Ω"/>
+<part name="R10" library="JBJLC" deviceset="RES_SMD" device="0805" value="60.4Ω"/>
 <part name="R8" library="JBJLC" deviceset="RES_SMD" device="0805" value="2.2kΩ"/>
 <part name="R7" library="JBJLC" deviceset="RES_SMD" device="0805" value="2.2kΩ"/>
